File: 3D_designs/Calibration Files/Alignment PCB/Alignment PCB.kicad_pcb (KiCad board)
At the start: 2 copper layers, 40 x 40 mm, 7 parts, among them J1 Conn_01x02_Socket

Commit message: small updates on aligment pcb, create files for producton
Parts:
- D2, D3, D4: value LED -> LED 2V 20mA
- R1, R2: footprint Resistor_THT:R_Axial_DIN0204_L3.6mm_D1.6mm_P7.62mm_Horizontal -> Resistor_THT:R_Axial_DIN0207_L6.3mm_D2.5mm_P7.62mm_Horizontal
Routing:
- net Net-(D3-K): track 31.1 -> 35.2 mm
- net Net-(D1-K): track 32.0 -> 30.3 mm
- net GND: track 24.0 -> 25.3 mm
